Commit message: camera

File: urdf/slrc_bot.urdf (robot description, URDF)
Before this commit: robot slrc_bot, 13 links, 12 joints
Links:
- added link camera_link, mass 1e-5; collision box size=0.01 0.01 0.01; visual box size=0.03 0.03 0.03
Joints:
- added joint camera_joint: type fixed, parent base_link, child camera_link, origin xyz=-0.095 0 0.045 rpy=0 0 0, axis 0 1 0

Commit message: camera tested

File: urdf/slrc_bot.urdf (robot description, URDF)
Before this commit: robot slrc_bot, 14 links, 13 joints
Joints:
- joint camera_joint: origin xyz=-0.095 0 0.045 rpy=0 0 0 -> xyz=-0.095 0 0.045 rpy=0 0 3.14159
